File: KiCAD/ESP32EvoPilotRemote/ESP32EvoPilotRemote.kicad_pcb (KiCad board)
At the start: 2 copper layers, 69.8 x 50.8 mm, 13 parts, among them J1 433 MHz Transmitter, J2 D24V10F5, J3 Power, J3-1 Ant, J3-2 433MHz Receiver, J4 CAN-Transceiver, J5 Ant., J6 Ant., Q1 BC547, U1 esp32_38_pins

Commit message: feat: Update KiCAD and ino
Parts:
- removed J1: 433 MHz Transmitter, Connector_PinHeader_2.54mm:PinHeader_1x04_P2.54mm_Vertical
- removed J2: D24V10F5, Connector_PinHeader_2.54mm:PinHeader_1x05_P2.54mm_Vertical
- removed J5: Ant., Connector_Pin:Pin_D1.0mm_L10.0mm
- added  : , MountingHole:MountingHole_3.2mm_M3, F.Cu at (69.8, 81.3)
- added  : , MountingHole:MountingHole_3.2mm_M3, F.Cu at (127.0, 81.3)
- added U2: StepDown LM2596, ESP32EvoPilotRemote:YAAJ_DCDC_StepDown_LM2596, F.Cu at (77.5, 73.7)
Routing:
- net +5V: track 102.2 -> 168.2 mm, vias 1 -> 2
- net Net-(U1-Pad31): track 56.4 -> 0.00 mm, vias 2 -> 0
- net Net-(D1-Pad1): track 55.1 -> 89.4 mm
- net GND: track 116.0 -> 142.6 mm
- net +3V3: track 93.0 -> 75.6 mm
- net Net-(J1-Pad4): track 7.62 -> 0.00 mm
Other:
- board size 69.8 x 50.8 mm -> 69.8 x 74.9 mm
