File: KiCAD/ESP32EvoPilotRemote/ESP32EvoPilotRemote.sch (KiCad schematic (older format))
At the start: 13 parts, among them J1 433 MHz Transmitter, J2 D24V10F5, J3 Power, J3-1 Ant, J3-2 433MHz Receiver, J4 CAN-Transceiver, J5 Ant., J6 Ant., Q1 BC547, U1 esp32_38_pins

Commit message: feat: Update KiCAD and ino
Parts:
- removed J1: 433 MHz Transmitter, Connector_PinHeader_2.54mm:PinHeader_1x04_P2.54mm_Vertical, symbol Connector_Generic:Conn_01x04
- removed J2: D24V10F5, Connector_PinHeader_2.54mm:PinHeader_1x05_P2.54mm_Vertical, symbol Connector_Generic:Conn_01x05
- removed J5: Ant., Connector_Pin:Pin_D1.0mm_L10.0mm, symbol Connector_Generic:Conn_01x01
- added U2: YAAJ_DCDC_StepDown_LM2596, ESP32EvoPilotRemote:YAAJ_DCDC_StepDown_LM2596, symbol ESP32EvoPilotRemote-rescue:YAAJ_DCDC_StepDown_LM2596
Connections:
- wire segments 68 -> 63
